File: circuit/MLX90393_board3/MLX90393_board3.kicad_sch (KiCad schematic)
At the start: 12 parts, among them J1 Conn_02x04_Odd_Even, Q1 BSS138, Q2 BSS138, U5 AP2112K-3.3

Commit message: refactored socketio
Connections:
- net +3.3V: now also D1.2 (A); no longer D1.1 (K)
- net GND: now also D1.1 (K); no longer D1.2 (A)
Other:
- moved on the sheet: D1
Changed lines of the file:
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@@
     )
   )
-  (symbol (lib_id "Device:LED") (at 224.79 119.38 0) (unit 1)
+  (symbol (lib_id "Device:LED") (at 224.79 119.38 180) (unit 1)
     (in_bom yes) (on_board yes) (dnp no) (fields_autoplaced)
-    (property "Reference" "D1" (at 223.2025 113.03 0)
+    (property "Reference" "D1" (at 226.3775 111.76 0)
       (effects (font (size 1.27 1.27)))
     )
-    (property "Value" "LED" (at 223.2025 115.57 0)
+    (property "Value" "LED" (at 226.3775 114.3 0)
       (effects (font (size 1.27 1.27)))
     )
